File: Senior Design/Senior Design.sch (KiCad schematic (older format))
At the start: 27 parts, among them U1 Raspberry_Pi_Zero_W, U2 AP1509, U3 TPA2005D1DRB, U4 ADC1210S21

Commit message: update
ddds
Parts:
- removed Conn1, Conn2: Molex_SL_04, MRDT_Connectors:MOLEX_SL_04_Horizontal, symbol MRDT_Connectors:Molex_SL_04
- added Conn1: Molex_SL_07, MRDT_Connectors:MOLEX_SL_07_Horizontal, symbol MRDT_Connectors:Molex_SL_07
- added Conn2: AndersonPP, MRDT_Connectors:Anderson_1_Horizontal, symbol MRDT_Connectors:AndersonPP
- C1, C5: value CP1 -> 10uF
- C3, C4, C6, C7: value 1u -> 1uF
- C8: value C_Small -> 1uF
- C9: value C_Small -> 0.1uF
Connections:
- net +3V3: no longer C5.1, C6.2, C7.2, C8.1, L1.2, R5.2, U2.3 (FB), U3.6 (VDD), U4.1 (Va)
- net GND: now also Conn1.1
- net IMU_SCL: now also Conn1.3
- net IMU_SDA: now also Conn1.2
- net LED_1: now also Conn1.7
- net LED_2: now also Conn1.6
- net LED_3: now also Conn1.5
- net Speak_OUT+: now also Conn3.2; no longer Conn3.1
- net Speak_OUT-: now also Conn3.1; no longer Conn3.2
- net +5V: now reaches U1.2 (5V)
- net +5V: now also C5.1, C6.2, C7.2, C8.1, L1.2, R5.2, U1.4 (5V), U2.3 (FB), U3.6 (VDD), U4.1 (Va), Conn1.4, Conn2.2 (V+Log)
- no-connect marks 24 -> 22
